File: MCU Datalogger.kicad_sch (KiCad schematic)
At the start: 25 parts, among them U1 DS1337S+, U2 24LC1025, U3 24LC1025, U4 ATMEGA328P-AU, Y1 32.768 KHz, Y2 16 MHz

Commit message: Small changes.
Connections:
- net Vcc: no longer U1.8 (VCC)
- net Abc123: no longer names the net of C4.2, U4.20 (AREF)
Changed lines of the file:
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@@
-	(wire
-		(pts
-			(xy 78.74 43.18) (xy 81.28 43.18)
-		)
-		(stroke
-			(width 0)
-			(type default)
-		)
-	)
 	(wire
 		(pts
@@
 	(label "Vcc"
 		(at 41.91 109.22 0)
-		(fields_autoplaced yes)
-		(effects
-			(font
-				(size 1.27 1.27)
-			)
-			(justify left bottom)
-		)
-	)
-	(label "Abc123"
-		(at 168.91 38.1 0)
 		(fields_autoplaced yes)
 		(effects
@@
 			)
 		)
+		(property "Purpose" ""
+			(at 157.48 38.1 0)
+			(effects
+				(font
+					(size 1.27 1.27)
+				)
+			)
+		)

Commit message: Fixed error with the I2C clock signal.
Connections:
- net SCK: no longer R3.2, U1.6 (SCL), U2.6 (SCL), U3.6 (SCL), U4.28 (PC5)
- net Vcc: now also U1.8 (VCC)
- net Abc123: now reaches C4.2, U4.20 (AREF)
- new net SCL: R3.2, U1.6 (SCL), U2.6 (SCL), U3.6 (SCL), U4.28 (PC5)
Other:
- sheet Connectors ports: added SCL; removed none
