File: MCU Datalogger.kicad_sch (KiCad schematic)
At the start: 25 parts, among them U1 DS1337S+, U2 24LC1025, U3 24LC1025, U4 ATMEGA328P-AU, Y1 32.768 KHz, Y2 16 MHz

Commit message: Fixed issue with I2C SCL signal.
Connections:
- net SCK: no longer R3.2, U1.6 (SCL), U2.6 (SCL), U3.6 (SCL), U4.28 (PC5)
- new net SCL: R3.2, U1.6 (SCL), U2.6 (SCL), U3.6 (SCL), U4.28 (PC5)
Other:
- sheet Connectors ports: added SCL; removed none
